File: MiniOSC.kicad_pcb (KiCad board)
At the start: 2 copper layers, 94.1 x 128.5 mm, 54 parts, among them J1 Conn_01x16_Female, J2 Conn_01x16_Male, J3 V_OCT_IN, J4 FM_IN, J5 PULSE_OUT, J6 SAW_OUT, J7 JST_BUS, J8 IDC_BUS, Q1 BC558, Q2 BC548, U1 TL074, U2 40106

Commit message: Added gerber files
Parts:
- added mouse-bite-2mm-slot: VAL**, Panelization:mouse-bite-2mm-slot, F.Cu at (71.0, 64.0)
- added mouse-bite-2mm-slot: VAL**, Panelization:mouse-bite-2mm-slot, F.Cu at (103.0, 64.0)
- moved mouse-bite-2mm-slot 13.2 mm to (71.0, 143.0)
- moved TUNING_FINE1 0.60 mm to (88.5, 95.0)
- moved FM_AMOUNT1 0.50 mm to (93.5, 102.0)
- moved J3 0.25 mm to (78.0, 134.0)
- moved J4 0.25 mm to (78.0, 114.5)
- moved J5 0.25 mm to (96.0, 149.5)
- moved J6 0.25 mm to (85.0, 149.4)
- moved PULSE_WIDTH1 0.25 mm to (88.5, 139.5)
- moved SCALE1 0.25 mm to (77.0, 158.2)
Routing:
- net /FrontPanel/FP_SAW_OUT: track 62.1 -> 65.9 mm
- net /FrontPanel/FP_PULSE_OUT: track 69.3 -> 72.7 mm
- net /FrontPanel/FP_V_OCT_IN: track 83.3 -> 85.4 mm
- net /FrontPanel/FP_PULSE_WIDTH: track 49.8 -> 51.7 mm
- net +12V: track 134.7 -> 134.0 mm
- net /FrontPanel/FP_COARSE: track 54.9 -> 54.3 mm
- net /FrontPanel/FP_FM_AMT_P3: track 17.8 -> 17.3 mm
- net /FrontPanel/FP_FM_AMT_P2: track 23.9 -> 23.4 mm
Other:
- outline, holes or cut-outs redrawn
- board text added: "@benjiaomodular"
- board text added: "MiniOSC (rev 1.0)"
- board text removed: "benjiaomodular"
