File: Fabrication/MiniOSC-rev1.2/MiniOSC - Main.kicad_pcb (KiCad board)
At the start: 2 copper layers, 94.1 x 128.5 mm, 54 parts, among them J1 Conn_01x16_Female, J2 Conn_01x16_Male, J3 V_OCT_IN, J4 FM_IN, J5 PULSE_OUT, J6 SAW_OUT, J7 JST_BUS, J8 IDC_BUS, Q1 BC558, Q2 BC548, U1 TL074, U2 40106

Commit message: Added v1.2
Parts:
- removed D3: LED, LED_THT:LED_D3.0mm
- removed FM_AMOUNT1: 1M, benjiaomodular:Potentiometer_RV09
- removed J2: Conn_01x16_Male, Connector_PinSocket_2.54mm:PinSocket_1x16_P2.54mm_Vertical
- removed J3: V_OCT_IN, Connector_Audio:Jack_3.5mm_QingPu_WQP-PJ398SM_Vertical_CircularHoles
- removed J4: FM_IN, Connector_Audio:Jack_3.5mm_QingPu_WQP-PJ398SM_Vertical_CircularHoles
- removed J5: PULSE_OUT, Connector_Audio:Jack_3.5mm_QingPu_WQP-PJ398SM_Vertical_CircularHoles
- removed J6: SAW_OUT, Connector_Audio:Jack_3.5mm_QingPu_WQP-PJ398SM_Vertical_CircularHoles
- removed PULSE_WIDTH1, TUNING_COARSE1, TUNING_FINE1: 100K, benjiaomodular:Potentiometer_RV09
- removed R18: 10K, Resistor_THT:R_Axial_DIN0207_L6.3mm_D2.5mm_P7.62mm_Horizontal
- removed the REF** at (47.5, 170.4)
- removed the REF** at (48.9, 48.0)
- removed the REF** at (94.8, 122.0)
- removed SCALE1: 1K, Potentiometer_THT:Potentiometer_Bourns_3266Y_Vertical
- removed TH2: 10K NTC, Capacitor_THT:C_Disc_D3.8mm_W2.6mm_P2.50mm
Routing:
- net /FrontPanel/FP_V_OCT_IN: track 85.4 -> 0.00 mm
- net /FrontPanel/FP_PULSE_OUT: track 72.7 -> 0.00 mm
- net /FrontPanel/FP_SAW_OUT: track 65.9 -> 0.00 mm
- net /FrontPanel/FP_SCALE: track 56.5 -> 0.00 mm
- net /FrontPanel/FP_COARSE: track 54.3 -> 0.00 mm
- net /FrontPanel/FP_PULSE_WIDTH: track 51.7 -> 0.00 mm
- net /FrontPanel/FP_FM_IN: track 46.1 -> 0.00 mm
- net FP_12V_NEG: track 39.9 -> 0.00 mm
- net /FrontPanel/FP_FM_AMT_P2: track 23.4 -> 0.00 mm
- net /FrontPanel/FP_FINE: track 21.6 -> 0.00 mm
- net /FrontPanel/FP_FM_AMT_P3: track 17.3 -> 0.00 mm
- net /FrontPanel/FP_12V_POS: track 16.8 -> 0.00 mm
- net Net-(D3-Pad2): track 7.59 -> 0.00 mm
- net GND1: vias 229 -> 0
- removed copper zone on B.Cu, net GND1
- removed copper zone on F.Cu, net GND1
Other:
- board size 94.1 x 128.5 mm -> 30.1 x 108.5 mm
- board text removed: "COARSE"
- board text removed: "FINE"
- board text removed: "FM AMOUNT"
- board text removed: "FM IN"
- board text removed: "M3 x 12mm standoff/spacer"
- board text removed: "MiniOSC"
- board text removed: "PULSE OUT"
- board text removed: "PULSE WIDTH"
- board text removed: "SAW OUT"
- board text removed: "SCALE"
- board text removed: "V/OCT"
