File: Fabrication/MiniOSC-rev1.2/MiniOSC - Main - BROKEN.kicad_pcb (KiCad board)
At the start: 2 copper layers, 30.1 x 108.5 mm, 39 parts, among them J1 Conn_01x16_Female, J7 JST_BUS, J8 IDC_BUS, Q1 BC558, Q2 BC548, U1 TL074, U2 40106

Commit message: Added updated build files for 1.2
Parts:
- removed TH2: 10K NTC, Capacitor_THT:C_Disc_D3.8mm_W2.6mm_P2.50mm
Other:
- board text added: "MiniOSC (rev 1.1.1)"
- board text removed: "M3 x 12mm standoff/spacer"
- board text removed: "MiniOSC (rev 1.2)"
