File: hardware/kicad/MiniOSC/MiniOSC.kicad_sch (KiCad schematic)
At the start: 63 parts, among them J10 FM_IN, J11 PWM_CV, J12 TRI_OUT, J13 SAW_OUT, J14 PULSE_OUT, J2 Conn_01x10_Pin, J9 VOCT_IN, Q3 BC848, Q4 BC858, U1 40106, U2 TL074, U3 TL074

Commit message: v2.0 PCB
Parts:
- added D1: 1N4148W, Diode_SMD:D_SOD-123, symbol Diode:1N4148W
- added J1: SYNC_IN, benjiaomodular:AudioJack_3.5mm, symbol benjiaomodular:PJ3001F
- added R19: 1k, Resistor_SMD:R_0603_1608Metric_Pad0.98x0.95mm_HandSolder, symbol Device:R
- added SW1: SW_DPDT_x2, benjiaomodular:Button_KFC7x7, symbol Switch:SW_DPDT_x2
- added TP6: TestPoint, Connector_Wire:SolderWirePad_1x01_SMD_1x2mm, symbol Connector:TestPoint
- C3, C4, C5, C6, C7: footprint Capacitor_SMD:C_0603_1608Metric_Pad1.08x0.95mm_HandSolder -> Capacitor_SMD:C_0805_2012Metric_Pad1.18x1.45mm_HandSolder
- J2: footprint Connector_IDC:IDC-Header_2x05_P2.54mm_Vertical -> benjiaomodular:Header_IDC2x05_NoArrow
- SCALE1: footprint benjiaomodular:Potentiometer_RV09 -> Potentiometer_THT:Potentiometer_Bourns_3266Y_Vertical
Connections:
- net GND: now also U2.5 (+), J1.S; no longer U3.13 (-)
- net at FM_AMT1.1, FM_AMT1.2, TH2.1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: now also Q4.1 (B), R5.2, TH3.1
- net at C8.1, D3.1 (K), Q3.3 (C)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: now also SW1.3 (C), TP6.1; no longer TP4.1
- net at C1.2, R11.2, TP5.1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: now also U2.12 (+), U3.10 (+); no longer U2.10 (+), U2.5 (+)
- net at R14.1, R16.1: now also U3.9 (-); no longer U2.6 (-)
- net at R16.2, R17.1: now also U3.8; no longer U2.7
- net at U2.8: now also R12.1, U2.9 (-); no longer R10.2
- net at R7.1, R8.1, R9.1: now also U2.13 (-); no longer U2.9 (-)
- net at R10.1, R24.1: now also U2.10 (+); no longer U2.12 (+)
- net at C2.2, R20.2: now also U3.12 (+); no longer U3.10 (+)
- net at R21.1, R22.1: now also U3.13 (-); no longer U3.9 (-)
- net at R22.2, R23.1: now also U3.14; no longer U3.8
- new net: U2.6 (-), U2.7
- new net: R10.2, U2.14
- new net: R19.1, SW1.2 (B)
- new net: D1.2 (A), J1.T
- new net: J1.TN, TP4.1
- new net: D1.1 (K), R19.2
- no-connect marks 8 -> 12
Other:
- moved on the sheet: C2, D2, D4, FM_AMT1, J10, J12, J9, Q3, Q4, R1, R13, R15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
