File: hardware/kicad/MiniOSC/MiniOSC.kicad_pcb (KiCad board)
At the start: 2 copper layers, 65 x 128.5 mm, 82 parts, among them J1 SYNC_IN, J10 FM_IN, J11 PWM_CV, J12 TRI_OUT, J13 SAW_OUT, J14 PULSE_OUT, J2 Conn_01x10_Pin, J9 VOCT_IN, Q3 BC848, Q4 BC858, SW1 SW_DPDT_x2, U1 40106, U2 TL074, U3 TL074

Commit message: Added fab files for v2.1
Parts:
- moved R8 1.43 mm to (179.8, 99.2), turned to 180 degrees
- moved R9 1.29 mm to (179.8, 97.7), turned to 180 degrees
- moved R7 0.81 mm to (182.3, 98.3), turned to 90 degrees
Routing:
- net Net-(FM_AMT1-Pad3): track 56.6 -> 53.9 mm
- net Net-(PULSE_WIDTH1-Pad2): track 18.4 -> 17.3 mm
- net Net-(R5-Pad1): track 7.59 -> 8.67 mm
- net Net-(U2D--): track 8.74 -> 9.64 mm
- net Net-(J10-PadT): track 62.6 -> 61.8 mm
- net Net-(PWM_AMT1-Pad1): track 28.0 -> 28.6 mm
- net Net-(D3-K): vias 4 -> 6
- net GND: vias 59 -> 69

Commit message: Updated R21 value
Parts:
- R21: value 10k -> 20k
Changed lines of the file:
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@@
 			)
 		)
-		(property "Value" "10k"
+		(property "Value" "20k"
 			(at 0 -1.43 0)
 			(layer "B.Fab")
