File: hardware/kicad/MiniOSC/MiniOSC.kicad_pcb (KiCad board)
At the start: 2 copper layers, 65 x 128.5 mm, 82 parts, among them J1 SYNC_IN, J10 FM_IN, J11 PWM_CV, J12 TRI_OUT, J13 SAW_OUT, J14 PULSE_OUT, J2 Conn_01x10_Pin, J9 VOCT_IN, Q3 BC848, Q4 BC858, SW1 SW_DPDT_x2, U1 40106, U2 TL074, U3 TL074

Commit message: Fixed typo on R14 value
Parts:
- R14: value 33k -> 68k
Changed lines of the file:
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@@
 	(title_block
 		(title "MiniOSC")
-		(rev "v2.1")
+		(rev "2.1")
 		(company "benjiaomodular")
 	)
@@
 			)
 		)
-		(property "Value" "33k"
+		(property "Value" "68k"
 			(at -0.1825 4.0125 0)
 			(layer "B.Fab")

Commit message: Added links to PCBWay, updated bom
Parts:
- C8: value 680pF -> 2.2nF
Changed lines of the file:
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@@
 			)
 		)
-		(property "Value" "680pF"
+		(property "Value" "2.2nF"
 			(at 3.6375 0 90)
 			(layer "B.Fab")
@@
 			)
 		)
-		(property "URL" "https://mou.sr/4goVMgC"
+		(property "URL" "https://mou.sr/3zee3wG"
 			(at 0 0 90)
 			(unlocked yes)
