File: hardware/legacy_versions/v1.2/kicad/MiniOSC 1.2/FrontPanel.kicad_sch (KiCad schematic)
At the start: 11 parts, among them J3 V_OCT_IN, J4 FM_IN, J5 PULSE_OUT, J6 SAW_OUT

Commit message: Added v2.1
Parts:
- gave numbers to parts that had none: 5
