File: hardware/legacy_versions/v2.0/kicad/MiniOSC/MiniOSC.kicad_pcb (KiCad board)
At the start: 2 copper layers, 65 x 128.5 mm, 82 parts, among them J1 SYNC_IN, J10 FM_IN, J11 PWM_CV, J12 TRI_OUT, J13 SAW_OUT, J14 PULSE_OUT, J2 Conn_01x10_Pin, J9 VOCT_IN, Q3 BC848, Q4 BC858, SW1 SW_DPDT_x2, U1 40106, U2 TL074, U3 TL074

Commit message: Added v2.1
Parts:
- C10, C9: footprint Capacitor_SMD:CP_Elec_4x5.8 -> Capacitor_SMD:CP_Elec_6.3x4.5
- C8: value 680pF -> 2.2nF
- SCALE1: footprint Potentiometer_THT:Potentiometer_Bourns_3296W_Vertical -> Potentiometer_THT:Potentiometer_Bourns_3266Y_Vertical
- moved PWM_AMT1 16.6 mm to (194.5, 95.5)
- moved PULSE_WIDTH1 16.6 mm to (196.1, 112.0)
- moved SCALE1 0.16 mm to (182.4, 93.9)
Routing:
- net Net-(J11-PadT): track 19.6 -> 36.4 mm
- net Net-(PULSE_WIDTH1-Pad2): track 18.4 -> 28.3 mm
- net Net-(J14-PadT): track 64.4 -> 73.2 mm
- net -12V: track 184.8 -> 191.2 mm
- net Net-(PWM_AMT1-Pad1): track 28.0 -> 21.7 mm
- net +12V: track 191.8 -> 198.1 mm
- net Net-(FM_AMT1-Pad3): track 56.6 -> 53.6 mm
- net Net-(U2D-+): track 107.9 -> 105.7 mm
- net GND: vias 59 -> 58
Other:
- outline, holes or cut-outs redrawn
- board text added: "MiniOSC v2.0"
- board text removed: "MiniOSC v2.1"
