File: hardware/legacy_versions/v2.0/kicad/MiniOSC/MiniOSC.kicad_sch (KiCad schematic)
At the start: 68 parts, among them J1 SYNC_IN, J10 FM_IN, J11 PWM_CV, J12 TRI_OUT, J13 SAW_OUT, J14 PULSE_OUT, J2 Conn_01x10_Pin, J9 VOCT_IN, Q3 BC848, Q4 BC858, SW1 SW_DPDT_x2, U1 40106, U2 TL074, U3 TL074

Commit message: Added v2.1
Parts:
- C10, C9: footprint Capacitor_SMD:CP_Elec_4x5.8 -> Capacitor_SMD:CP_Elec_6.3x4.5
- C8: value 680pF -> 2.2nF
- SCALE1: footprint Potentiometer_THT:Potentiometer_Bourns_3296W_Vertical -> Potentiometer_THT:Potentiometer_Bourns_3266Y_Vertical; URL https://www.taydaelectronics.com/1k-ohm-trimmer-potentiomet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 -> https://mou.sr/3MFeCCP
Changed lines of the file:
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@@
 	(title_block
 		(title "MiniOSC")
-		(rev "2.1")
+		(rev "2.0")
 		(company "benjiaomodular")
 	)
@@
 			)
 		)
-		(property "Value" "680pF"
+		(property "Value" "2.2nF"
 			(at 122.301 59.563 0)
 			(effects
@@
 			)
 		)
-		(property "Footprint" "Capacitor_SMD:CP_Elec_4x5.8"
+		(property "Footprint" "Capacitor_SMD:CP_Elec_6.3x4.5"
 			(at 51.7652 165.1 0)
 			(effects
@@
 			)
 		)
-		(property "Footprint" "Capacitor_SMD:CP_Elec_4x5.8"
+		(property "Footprint" "Capacitor_SMD:CP_Elec_6.3x4.5"
 			(at 51.7652 177.8 0)
 			(effects
@@
 			)
 		)
-		(property "Footprint" "Potentiometer_THT:Potentiometer_Bourns_3296W_Vertical"
+		(property "Footprint" "Potentiometer_THT:Potentiometer_Bourns_3266Y_Vertical"
 			(at 75.692 82.55 90)
 			(effects
@@
 			)
 		)
-		(property "URL" "https://www.taydaelectronics.com/1k-ohm-trimmer-potentiometer-cermet-25-turns-3296w.html"
+		(property "URL" "https://mou.sr/3MFeCCP"
 			(at 77.47 82.55 0)
 			(effects
